File: Hardware/BME280_Breakout.brd (EAGLE design)
At the start: 12.7 x 20.3 mm, 20 parts, among them U1 BME280

Commit message: ready for QC check
Parts:
- SJ1: value (none) -> EN I2C PULL
- SJ2: value JUMPER-PAD-2-NC_BY_TRACE -> EN SPI CS
- SJ3: value JUMPER-PAD-3-2OF3_NC_BY_PASTE -> EN ADR PULLUP
Other:
- board text added: "Marshall Taylor"
Changed lines of the file:
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@@
 <text x="7.3025" y="2.54" size="0.8128" layer="22" font="vector" ratio="15" rot="MR0" align="center-left">PULL_EN</text>
 <text x="8.5328125" y="1.8653125" size="1.27" layer="16" font="vector" ratio="15" rot="MR180">v01</text>
+<text x="5.08" y="-22.86" size="1.778" layer="51">Marshall Taylor</text>
 </plain>
 <attributes>
@@
 <attribute name="PROD_ID" value="RES-07857" x="6.985" y="16.8275" size="1.778" layer="27" display="off"/>
 </element>
-<element name="SJ1" library="SparkFun-Passives" package="PAD-JUMPER-3-3OF3_NC_BY_TRACE_YES_SILK_FULL_BOX" value="" x="3.175" y="5.08" rot="MR90"/>
-<element name="SJ2" library="SparkFun-Passives" package="PAD-JUMPER-2-NC_BY_TRACE_YES_SILK" value="JUMPER-PAD-2-NC_BY_TRACE" x="7.3025" y="5.3975" rot="MR270"/>
-<element name="SJ3" library="SparkFun-Passives" package="PAD-JUMPER-3-2OF3_NC_BY_PASTE_YES_SILK_FULL_BOX" value="JUMPER-PAD-3-2OF3_NC_BY_PASTE" x="2.619375" y="19.20875"/>
+<element name="SJ1" library="SparkFun-Passives" package="PAD-JUMPER-3-3OF3_NC_BY_TRACE_YES_SILK_FULL_BOX" value="EN I2C PULL" x="3.175" y="5.08" rot="MR90"/>
+<element name="SJ2" library="SparkFun-Passives" package="PAD-JUMPER-2-NC_BY_TRACE_YES_SILK" value="EN SPI CS" x="7.3025" y="5.3975" rot="MR270"/>
+<element name="SJ3" library="SparkFun-Passives" package="PAD-JUMPER-3-2OF3_NC_BY_PASTE_YES_SILK_FULL_BOX" value="EN ADR PULLUP" x="2.619375" y="19.20875"/>
 <element name="U1" library="BME280ComponentLibrary" package="BME280_LGA" value="BME280" x="6.35" y="10.16" rot="R270">
 <attribute name="PROD_ID" value="IC-13090" x="6.35" y="10.16" size="1.778" layer="27" rot="R270" display="off"/>
