File: Hardware/BME280_Breakout.brd (EAGLE design)
At the start: 12.7 x 20.3 mm, 19 parts, among them U1 BME280

Commit message: Ready for review
Parts:
- SJ2: value EN SPI CS -> EN I2C MODE
Connections:
- net 3.3V: now also JP2.5; no longer JP2.6
- net GND: now also JP2.6; no longer JP2.5
Routing:
- net N$1: track 4.68 -> 3.34 mm
- net N$2: track 4.68 -> 3.45 mm
Other:
- board text added: "CS PU"
- board text added: "I2C PU"
- board text removed: "ENB P-UP"
