File: Hardware/BME280_Breakout.sch (EAGLE design)
At the start: 11 parts, among them U1 BME280

Commit message: Pre-checklist commit
Parts:
- added FID1, FID2: FIDUCIAL1X2, SparkFun-Aesthetics:FIDUCIAL1X2
- added JP1: (no value), SparkFun-Connectors:I2C_STANDARD_NO_SILK
- added JP2: (no value), SparkFun-Connectors:M06NO_SILK_FEMALE_PTH
- added LOGO1: SFE_LOGO_NAME.1_INCH, SparkFun-Aesthetics:SFE_LOGO_NAME.1_INCH
- added LOGO2: SFE_LOGO_FLAME.1_INCH, SparkFun-Aesthetics:SFE_LOGO_FLAME.1_INCH
- added LOGO3: OSHW-LOGOS, SparkFun-Aesthetics:OSHW-LOGOS
- added STANDOFF1, STANDOFF4: STAND-OFF, SparkFun-Electromechanical:STAND-OFF
Connections:
- net !CS: now also JP2.1
- net 3.3V: now also JP1.2, JP2.6
- net GND: now also JP1.1, JP2.5
- net SCK/SCL: now also JP1.4, JP2.4
- net SDI/SDA: now also JP1.3, JP2.2
- net SDO/ADR: now also JP2.3
Other:
- note added: "(Use only 1)"
- note added: "BME280 Breakout"
- note added: "I2C"
- note added: "Marshall Taylor"
- note added: "Ports:"
- note added: "SJ1 and SJ2 allow disconnection of the pull-up resistors. Disconnect for SPI mode if necessary."
- note added: "SJ3 controls the lowest bit of the I2C address. Open for SPI mode"
- note added: "SPI"
- note added: "V01"
- moved on the sheet: C1, C2, R1, R2, R3, R4, SJ1, SJ2, SJ3, U1

Commit message: ready for QC check
Parts:
- SJ1: value (none) -> EN I2C PULL
- SJ2: value JUMPER-PAD-2-NC_BY_TRACE -> EN SPI CS
- SJ3: value JUMPER-PAD-3-2OF3_NC_BY_PASTE -> EN ADR PULLUP
Other:
- note added: "SJ3 controls the lowest bit of the I2C address--can be: 0x1110110 0x1110111 Open for SPI mode"
- note removed: "SJ3 controls the lowest bit of the I2C address. Open for SPI mode"
Changed lines of the file:
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@@
 <part name="C1" library="SparkFun-Capacitors" deviceset="0.1UF-25V-5%(0603)" device="" value="0.1uF"/>
 <part name="C2" library="SparkFun-Capacitors" deviceset="0.1UF-25V-5%(0603)" device="" value="0.1uF"/>
-<part name="SJ1" library="SparkFun-Passives" deviceset="JUMPER-PAD-3-NC_BY_TRACE" device=""/>
+<part name="SJ1" library="SparkFun-Passives" deviceset="JUMPER-PAD-3-NC_BY_TRACE" device="" value="EN I2C PULL"/>
 <part name="SUPPLY3" library="SparkFun-Aesthetics" deviceset="3.3V" device=""/>
 <part name="R1" library="SparkFun-Resistors" deviceset="4.7KOHM-1/10W-1%(0603)" device="" value="4.7K"/>
 <part name="R2" library="SparkFun-Resistors" deviceset="4.7KOHM-1/10W-1%(0603)" device="" value="4.7K"/>
 <part name="R3" library="SparkFun-Resistors" deviceset="4.7KOHM-1/10W-1%(0603)" device="" value="4.7K"/>
-<part name="SJ2" library="SparkFun-Passives" deviceset="JUMPER-PAD-2-NC_BY_TRACE" device=""/>
+<part name="SJ2" library="SparkFun-Passives" deviceset="JUMPER-PAD-2-NC_BY_TRACE" device="" value="EN SPI CS"/>
 <part name="SUPPLY4" library="SparkFun-Aesthetics" deviceset="3.3V" device=""/>
-<part name="SJ3" library="SparkFun-Passives" deviceset="JUMPER-PAD-3-2OF3_NC_BY_PASTE" device=""/>
+<part name="SJ3" library="SparkFun-Passives" deviceset="JUMPER-PAD-3-2OF3_NC_BY_PASTE" device="" value="EN ADR PULLUP"/>
 <part name="R4" library="SparkFun-Resistors" deviceset="4.7KOHM-1/10W-1%(0603)" device="" value="4.7K"/>
 <part name="SUPPLY5" library="SparkFun-Aesthetics" deviceset="3.3V" device=""/>
@@
 <text x="236.728" y="6.604" size="2.54" layer="94">V01</text>
 <text x="7.62" y="172.72" size="3.81" layer="97">BME280 Breakout</text>
-<text x="10.668" y="131.318" size="1.778" layer="97" align="top-left">SJ3 controls the lowest bit
-of the I2C address.
-Open for SPI mode</text>
+<text x="8.128" y="141.478" size="1.778" layer="97" align="top-left">SJ3 controls the lowest bit
+of the I2C address--can be:
+  0x1110110
+  0x1110111
+  Open for SPI mode</text>
 <text x="145.288" y="166.878" size="1.778" layer="97" align="top-left">SJ1 and SJ2 allow disconnection of the
 pull-up resistors.  Disconnect for SPI
 mode if necessary.</text>
 <text x="7.62" y="55.88" size="3.81" layer="97">Ports:</text>
-<wire x1="248.92" y1="66.04" x2="147.32" y2="66.04" width="0.1524" layer="94"/>
-<wire x1="147.32" y1="66.04" x2="0" y2="66.04" width="0.1524" layer="94"/>
-<wire x1="147.32" y1="35.56" x2="147.32" y2="66.04" width="0.1524" layer="94"/>
+<wire x1="248.92" y1="66.04" x2="147.32" y2="66.04" width="0.1524" layer="97" style="longdash"/>
+<wire x1="147.32" y1="66.04" x2="0" y2="66.04" width="0.1524" layer="97" style="longdash"/>
+<wire x1="147.32" y1="35.56" x2="147.32" y2="66.04" width="0.1524" layer="97" style="longdash"/>
 <text x="8.128" y="53.848" size="1.778" layer="97" align="top-left">(Use only 1)</text>
 <text x="27.94" y="41.148" size="3.81" layer="97">I2C</text>
@@
 <instance part="C1" gate="G$1" x="86.36" y="96.52"/>
 <instance part="C2" gate="G$1" x="93.98" y="96.52"/>
-<instance part="SJ1" gate="G$1" x="154.94" y="139.7" rot="R270"/>
+<instance part="SJ1" gate="G$1" x="154.94" y="139.7" smashed="yes" rot="R270">
+<attribute name="NAME" x="152.781" y="137.16" size="1.778" layer="95" rot="R270"/>
+<attribute name="VALUE" x="155.575" y="137.16" size="1.778" layer="96" rot="R270"/>
+</instance>
 <instance part="SUPPLY3" gate="G$1" x="154.94" y="147.32"/>
 <instance part="R1" gate="G$1" x="147.32" y="132.08" rot="R90"/>
@@
 <instance part="R3" gate="G$1" x="177.8" y="124.46" rot="R90"/>
 <instance part="SJ2" gate="G$1" x="177.8" y="137.16" smashed="yes" rot="R90">
-<attribute name="NAME" x="175.26" y="134.62" size="1.778" layer="95" rot="R90"/>
+<attribute name="NAME" x="180.34" y="142.24" size="1.778" layer="95" rot="R270"/>
+<attribute name="VALUE" x="182.88" y="142.24" size="1.778" layer="96" rot="R270"/>
 </instance>
 <instance part="SUPPLY4" gate="G$1" x="177.8" y="147.32"/>
 <instance part="SJ3" gate="G$1" x="58.42" y="124.46" smashed="yes" rot="R180">
-<attribute name="NAME" x="55.88" y="124.079" size="1.778" layer="95" rot="R180"/>
+<attribute name="NAME" x="52.959" y="121.92" size="1.778" layer="95" rot="R90"/>
+<attribute name="VALUE" x="55.245" y="121.92" size="1.778" layer="96" rot="R90"/>
 </instance>
 <instance part="R4" gate="G$1" x="58.42" y="137.16" rot="R90"/>
@@
 </sheet>
 </sheets>
+<errors>
+</errors>
 </schematic>
 </drawing>

Commit message: Rev 0.2
Parts:
- removed STANDOFF1: STAND-OFF, SparkFun-Electromechanical:STAND-OFF
- LOGO1: value SFE_LOGO_NAME.1_INCH -> SFE_LOGO_FLAME.1_INCH; device SparkFun-Aesthetics:SFE_LOGO_NAME.1_INCH -> SparkFun-Aesthetics:SFE_LOGO_FLAME.1_INCH
- SJ3: device SparkFun-Passives:JUMPER-PAD-3-2OF3_NC_BY_PASTE -> SparkFun-Passives:JUMPER-PAD-3-2OF3_NC_BY_TRACE_SMALL
Other:
- note added: "Note: Can be left connected for SPI at the cost of an extra 4.7k Ohm loading during data '0's"
- note added: "V02"
- note removed: "V01"
Changed lines of the file:
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@@
 <part name="SJ2" library="SparkFun-Passives" deviceset="JUMPER-PAD-2-NC_BY_TRACE" device="" value="EN SPI CS"/>
 <part name="SUPPLY4" library="SparkFun-Aesthetics" deviceset="3.3V" device=""/>
-<part name="SJ3" library="SparkFun-Passives" deviceset="JUMPER-PAD-3-2OF3_NC_BY_PASTE" device="" value="EN ADR PULLUP"/>
+<part name="SJ3" library="SparkFun-Passives" deviceset="JUMPER-PAD-3-2OF3_NC_BY_TRACE" device="_SMALL" value="EN ADR PULLUP"/>
 <part name="R4" library="SparkFun-Resistors" deviceset="4.7KOHM-1/10W-1%(0603)" device="" value="4.7K"/>
 <part name="SUPPLY5" library="SparkFun-Aesthetics" deviceset="3.3V" device=""/>
 <part name="GND5" library="SparkFun-Aesthetics" deviceset="GND" device=""/>
-<part name="STANDOFF1" library="SparkFun-Electromechanical" deviceset="STAND-OFF" device=""/>
 <part name="STANDOFF4" library="SparkFun-Electromechanical" deviceset="STAND-OFF" device=""/>
 <part name="FID1" library="SparkFun-Aesthetics" deviceset="FIDUCIAL" device="1X2"/>
@@
 <part name="GND7" library="SparkFun-Aesthetics" deviceset="GND" device=""/>
 <part name="SUPPLY7" library="SparkFun-Aesthetics" deviceset="3.3V" device=""/>
-<part name="LOGO1" library="SparkFun-Aesthetics" deviceset="SFE_LOGO_NAME" device=".1_INCH"/>
+<part name="LOGO1" library="SparkFun-Aesthetics" deviceset="SFE_LOGO_FLAME" device=".1_INCH" value="SFE_LOGO_FLAME.1_INCH"/>
 <part name="LOGO2" library="SparkFun-Aesthetics" deviceset="SFE_LOGO_FLAME" device=".1_INCH"/>
 <part name="LOGO3" library="SparkFun-Aesthetics" deviceset="OSHW-LOGO" device="S"/>
@@
 <plain>
 <text x="171.704" y="11.43" size="2.54" layer="94">Marshall Taylor</text>
-<text x="236.728" y="6.604" size="2.54" layer="94">V01</text>
+<text x="236.728" y="6.604" size="2.54" layer="94">V02</text>
 <text x="7.62" y="172.72" size="3.81" layer="97">BME280 Breakout</text>
-<text x="8.128" y="141.478" size="1.778" layer="97" align="top-left">SJ3 controls the lowest bit
+<text x="5.588" y="141.478" size="1.778" layer="97" align="top-left">SJ3 controls the lowest bit
 of the I2C address--can be:
   0x1110110
@@
 <text x="27.94" y="41.148" size="3.81" layer="97">I2C</text>
 <text x="81.28" y="46.228" size="3.81" layer="97">SPI</text>
+<text x="5.588" y="126.238" size="1.778" layer="97" align="top-left">Note:
+  Can be left connected for
+  SPI at the cost of an extra
+  4.7k Ohm loading during
+  data '0's</text>
 </plain>
 <instances>
@@
 <instance part="SUPPLY5" gate="G$1" x="58.42" y="144.78"/>
 <instance part="GND5" gate="1" x="58.42" y="114.3"/>
-<instance part="STANDOFF1" gate="G$1" x="246.38" y="27.94"/>
-<instance part="STANDOFF4" gate="G$1" x="246.38" y="25.4"/>
+<instance part="STANDOFF4" gate="G$1" x="243.84" y="25.4"/>
 <instance part="FID1" gate="G$1" x="238.76" y="25.4"/>
 <instance part="FID2" gate="G$1" x="236.22" y="25.4"/>
@@
 <instance part="GND7" gate="1" x="111.76" y="15.24"/>
 <instance part="SUPPLY7" gate="G$1" x="111.76" y="45.72"/>
-<instance part="LOGO1" gate="G$1" x="149.606" y="40.132"/>
-<instance part="LOGO2" gate="G$1" x="212.598" y="43.18"/>
-<instance part="LOGO3" gate="G$1" x="233.68" y="48.26"/>
+<instance part="LOGO1" gate="G$1" x="160.528" y="43.18"/>
+<instance part="LOGO2" gate="G$1" x="187.198" y="43.18"/>
+<instance part="LOGO3" gate="G$1" x="220.98" y="50.8"/>
 </instances>
 <busses>

Commit message: Ready for review
Parts:
- SJ2: value EN SPI CS -> EN I2C MODE
Connections:
- net 3.3V: now also JP2.5; no longer JP2.6
- net GND: now also JP2.6; no longer JP2.5
Other:
- note added: "MODES: I2C: Leave the copper-connected jumpers SJ1-SJ2 as default, use SJ3 to set the I2C address. SPI 4-WIRE: Jumpers SJ1-SJ3 can be opened to remove 4.7k load on the SPI lines but is not necessary. SPI 3-WIRE: SJ3 must be opened."
- note added: "SJ1 pulls up the SCK and SDA lines for I2C operation"
- note added: "SJ2 pulls up the !CS! line forcing I2C mode if no signal is on !CS!."
- note added: "SJ3 controls the lowest bit of the I2C address--can be: 0x1110110 0x1110111 Open for SPI 3-wire mode"
- note removed: "Note: Can be left connected for SPI at the cost of an extra 4.7k Ohm loading during data '0's"
- note removed: "SJ1 and SJ2 allow disconnection of the pull-up resistors. Disconnect for SPI mode if necessary."
- note removed: "SJ3 controls the lowest bit of the I2C address--can be: 0x1110110 0x1110111 Open for SPI mode"
- moved on the sheet: C1, C2, R1, R2, R3, R4, SJ1, SJ2, SJ3, U1

Commit message: incremented version number
Other:
- note added: "V10"
- note removed: "V02"
Changed lines of the file:
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@@
 <plain>
 <text x="171.704" y="11.43" size="2.54" layer="94">Marshall Taylor</text>
-<text x="236.728" y="6.604" size="2.54" layer="94">V02</text>
+<text x="236.728" y="6.604" size="2.54" layer="94">V10</text>
 <text x="7.62" y="175.26" size="3.81" layer="97">BME280 Breakout</text>
 <text x="5.588" y="118.618" size="1.778" layer="97" align="top-left">SJ3 controls the lowest bit
